Commit message: Update inspire_hand_left.urdf
with meshes

File: urdf/inspire_hand_left.urdf (robot description, URDF)
Before this commit: robot inspire_hand_left, 19 links, 18 joints
Links:
- link hand_base_link: geometry collision box size=0.0125 0.0111 0.0089; collision box size=0.0125 0.0111 0.0089
- link index_intermediate: geometry collision mesh filename=package://inspire_hand/meshes/collision/left_index_intermed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; visual mesh filename=package://inspire_hand/meshes/visual/left_index_intermediat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
- link index_proximal: geometry collision mesh filename=package://inspire_hand/meshes/collision/left_index_proximal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; visual mesh filename=package://inspire_hand/meshes/visual/left_index_proximal.glb
- link middle_intermediate: geometry collision mesh filename=package://inspire_hand/meshes/collision/left_middle_interme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; visual mesh filename=package://inspire_hand/meshes/visual/left_middle_intermedia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
- link middle_proximal: geometry collision mesh filename=package://inspire_hand/meshes/collision/left_index_proximal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; visual mesh filename=package://inspire_hand/meshes/visual/left_index_proximal.glb
- link pinky_intermediate: geometry collision mesh filename=package://inspire_hand/meshes/collision/left_pinky_intermed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; visual mesh filename=package://inspire_hand/meshes/visual/left_pinky_intermediat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
- link pinky_proximal: geometry collision mesh filename=package://inspire_hand/meshes/collision/left_index_proximal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; visual mesh filename=package://inspire_hand/meshes/visual/left_index_proximal.glb
- link ring_intermediate: geometry collision mesh filename=package://inspire_hand/meshes/collision/left_index_intermed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; visual mesh filename=package://inspire_hand/meshes/visual/left_index_intermediat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
- link ring_proximal: geometry collision mesh filename=package://inspire_hand/meshes/collision/left_index_proximal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; visual mesh filename=package://inspire_hand/meshes/visual/left_index_proximal.glb
- link thumb_distal: geometry collision mesh filename=package://inspire_hand/meshes/collision/left_thumb_distal.o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 scale=1 1 1; visual mesh filename=package://inspire_hand/meshes/visual/left_thumb_distal.glb
- link thumb_intermediate: geometry collision mesh filename=package://inspire_hand/meshes/collision/left_thumb_intermed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; visual mesh filename=package://inspire_hand/meshes/visual/left_thumb_intermediat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
- link thumb_proximal: geometry collision mesh filename=package://inspire_hand/meshes/collision/left_thumb_proximal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; visual mesh filename=package://inspire_hand/meshes/visual/left_thumb_proximal.glb
- link thumb_proximal_base: geometry collision mesh filename=package://inspire_hand/meshes/collision/left_thumb_proximal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; visual mesh filename=package://inspire_hand/meshes/visual/left_thumb_proximal_ba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
